Commit message: Increase base mass further
Tweak some inertias
Note some candidate simplified wheel collision shapes for testing

File: stretch_description/urdf/stretch_main.xacro (robot description, xacro)
@@ -13,12 +13,12 @@
         rpy="0 0 0" />
       <mass
-        value="6.0" />
-      <inertia
-        ixx="0.00310580907710135"
-        ixy="1.5182848191076E-06"
-        ixz="0.00041690466732394"
-        iyy="0.00433798719991832"
-        iyz="1.33487716258445E-05"
-        izz="0.0037204727467362" />
+        value="12.0" />
+      <inertia
+        ixx="0.00013"
+        ixy="0"
+        ixz="0"
+        iyy="0.00012"
+        iyz="0"
+        izz="0.000218" />
     </inertial>
     <visual>
@@ -83,4 +83,5 @@
         <mesh
           filename="package://stretch_description/meshes/link_right_wheel.STL" />
+          <!-- <cylinder radius="0.051" length="0.0225" /> -->
       </geometry>
     </collision>
@@ -137,4 +138,5 @@
         <mesh
           filename="package://stretch_description/meshes/link_left_wheel.STL" />
+        <!-- <cylinder radius="0.051" length="0.0225" /> -->
       </geometry>
     </collision>
@@ -207,15 +209,15 @@
     <inertial>
       <origin
-        xyz="0.00755818572975822 0.773971284176834 0.00647313086620024"
+        xyz="0 0.7073971284176834 0"
         rpy="0 0 0" />
       <mass
         value="0.749143203376401" />
       <inertia
-        ixx="0.0709854511954588"
-        ixy="-0.00433428742758457"
-        ixz="-0.000186110788697573"
-        iyy="0.000437922053342648"
-        iyz="-0.00288788257713431"
-        izz="0.071104808501661" />
+        ixx="0.000251"
+        ixy="0"
+        ixz="-0"
+        iyy="0.000000"
+        iyz="0"
+        izz="0.000251" />
     </inertial>
     <visual>

Commit message: Add friction and damping to arm and lift joints
Friction keeps the lift joint from slamming down too easily

File: stretch_description/urdf/stretch_main.xacro (robot description, xacro)
@@ -3,5 +3,7 @@
   <xacro:property name="M_PI" value="3.1415926535897931" />
   <xacro:property name="joint_damping" value="21.75"/>
+  <xacro:property name="arm_damping" value="21.75"/>
   <xacro:property name="joint_friction" value="10.48"/>
+  <xacro:property name="arm_friction" value="2.48"/>
   <xacro:property name="joint_spring_stiffness" value="0"/>
   <xacro:property name="joint_spring_reference" value="0"/>
@@ -313,5 +315,6 @@
   <!--<limit effort="100" lower="0.0" upper="1.095" velocity="1.0"/>-->
   <!-- copied value did not reach the top of mesh model with GUI sliders and RViz -->
-  <limit effort="100" lower="0.0" upper="1.1" velocity="1.0"/>
+  <limit effort="100" lower="0.0" upper="1.1" velocity="0.5"/>
+  <dynamics friction="40.0" damping="5.0"/>
   </joint>
   <link
@@ -367,4 +370,5 @@
     <axis
       xyz="0 0 0" />
+    <dynamics damping="${arm_damping}" friction="${arm_friction}" />
   </joint>
   <link
@@ -421,5 +425,6 @@
 	xyz="0 0 1" />
     <!-- 0.13 = 0.52/4-->
-    <limit effort="100" lower="0.0" upper="0.13" velocity="1.0"/>
+    <limit effort="100" lower="0.0" upper="0.13" velocity="0.1"/>
+    <dynamics damping="${arm_damping}" friction="${arm_friction}" />
   </joint>
   <link
@@ -476,5 +481,6 @@
 	xyz="0 0 1" />
     <!-- 0.13 = 0.52/4-->
-    <limit effort="100" lower="0.0" upper="0.13" velocity="1.0"/>
+    <limit effort="100" lower="0.0" upper="0.13" velocity="0.1"/>
+    <dynamics damping="${arm_damping}" friction="${arm_friction}" />
   </joint>
   <link
@@ -531,5 +537,6 @@
 	xyz="0 0 1" />
     <!-- 0.13 = 0.52/4-->
-    <limit effort="100" lower="0.0" upper="0.13" velocity="1.0"/>
+    <limit effort="100" lower="0.0" upper="0.13" velocity="0.1"/>
+    <dynamics damping="${arm_damping}" friction="${arm_friction}" />
   </joint>
   <link
@@ -586,5 +593,6 @@
 	xyz="0 0 1" />
     <!-- 0.13 = 0.52/4-->
-    <limit effort="100" lower="0.0" upper="0.13" velocity="1.0"/>
+    <limit effort="100" lower="0.0" upper="0.13" velocity="0.1"/>
+    <dynamics damping="${arm_damping}" friction="${arm_friction}" />
   </joint>
   <link
@@ -646,5 +654,5 @@
       using -1.75
     -->
-    <limit effort="100" lower="-1.75" upper="4.0" velocity="1.0"/>
+    <limit effort="100" lower="-1.75" upper="4.0" velocity="0.3"/>
   </joint>
   <link
