Commit message: Add collision geometry and color matched materials
Round poses down to 0 if a value is less than 0.00001
Move stretch.xacro into a robots folder, per convention

File: stretch_description/urdf/stretch_gripper.xacro (robot description, xacro)
@@ -29,14 +29,22 @@
         name="">
         <color
-          rgba="0.792156862745098 0.819607843137255 0.933333333333333 1" />
-      </material>
-    </visual>
-    <collision>
-      <origin
-        xyz="0 0 0"
-        rpy="0 0 0" />
-      <geometry>
-        <mesh
-          filename="package://stretch_description/meshes/link_gripper.STL" />
+          rgba=".13 .13 .16 1" />
+      </material>
+    </visual>
+    <collision>
+      <origin
+        xyz="0 0 0"
+        rpy="0 0 0" />
+      <geometry>
+        <mesh
+          filename="package://stretch_description/meshes/collision/link_gripper.STL" />
+      </geometry>
+    </collision>
+    <collision>
+      <origin
+        xyz="-0.0039 0.0139 -0.0289"
+        rpy="0 0 0" />
+      <geometry>
+        <box size="0.0423 0.0618 0.0578" />
       </geometry>
     </collision>
@@ -49,5 +57,5 @@
     <origin
       xyz="0 0 0"
-      rpy="3.14159 0 -1.5708" />
+      rpy="3.14159 0 -${pi/2}" />
     <parent
       link="link_wrist_yaw" />
@@ -61,5 +69,5 @@
     <inertial>
       <origin
-        xyz="0.0945047483510102 0.0124301080924361 -4.44089209850063E-16"
+        xyz="0.0945047483510102 0.0124301080924361 0"
         rpy="0 0 0" />
       <mass
@@ -84,5 +92,5 @@
         name="">
         <color
-          rgba="0.792156862745098 0.819607843137255 0.933333333333333 1" />
+          rgba="0.8 .8 .8 1" />
       </material>
     </visual>
@@ -102,5 +110,5 @@
     <origin
       xyz="-0.047231 -0.010151 -0.04679"
-      rpy="2.1762E-15 0.5236 3.1416" />
+      rpy="0 0.5236 3.1416" />
     <parent
       link="link_gripper" />
@@ -115,5 +123,5 @@
     <inertial>
       <origin
-        xyz="-3.16381381648689E-08 -2.91408530639359E-09 0.00812579670381812"
+        xyz="0 0 0.00812579670381812"
         rpy="0 0 0" />
       <mass
@@ -133,19 +141,19 @@
       <geometry>
         <mesh
-          filename="package://stretch_description/meshes/link_gripper_fingertip_left.STL" />
-      </geometry>
-      <material
-        name="">
-        <color
-          rgba="0.250980392156863 0.250980392156863 0.250980392156863 1" />
-      </material>
-    </visual>
-    <collision>
-      <origin
-        xyz="0 0 0"
-        rpy="0 0 0" />
-      <geometry>
-        <mesh
-          filename="package://stretch_description/meshes/link_gripper_fingertip_left.STL" />
+          filename="package://stretch_description/meshes/link_gripper_fingertip.STL" />
+      </geometry>
+      <material
+        name="">
+        <color
+          rgba="0.25 0.25 0.25 1" />
+      </material>
+    </visual>
+    <collision>
+      <origin
+        xyz="0 0 0"
+        rpy="0 0 0" />
+      <geometry>
+        <mesh
+          filename="package://stretch_description/meshes/collision/link_gripper_fingertip.STL" />
       </geometry>
     </collision>
@@ -156,5 +164,5 @@
     <origin
       xyz="${scale_finger_length * 0.19011} 0.014912 0"
-      rpy="-1.5708 -4.774E-15 -2.5545" />
+      rpy="-${pi/2} 0 -2.5545" />
     <parent
       link="link_gripper_finger_left" />
@@ -191,5 +199,5 @@
         name="">
         <color
-          rgba="0.792156862745098 0.819607843137255 0.933333333333333 1" />
+          rgba=".8 .8 .8 1" />
       </material>
     </visual>
@@ -209,5 +217,5 @@
     <origin
       xyz="-0.047231 0.010049 -0.04679"
-      rpy="3.1416 -0.5236 1.2943E-15" />
+      rpy="3.1416 -0.5236 0" />
     <parent
       link="link_gripper" />
@@ -222,5 +230,5 @@
     <inertial>
       <origin
-        xyz="2.59386303963494E-08 6.70949018566347E-09 0.00812579516130402"
+        xyz="0 0 0.00812579516130402"
         rpy="0 0 0" />
       <mass
@@ -240,19 +248,19 @@
       <geometry>
         <mesh
-          filename="package://stretch_description/meshes/link_gripper_fingertip_right.STL" />
-      </geometry>
-      <material
-        name="">
-        <color
-          rgba="0.250980392156863 0.250980392156863 0.250980392156863 1" />
-      </material>
-    </visual>
-    <collision>
-      <origin
-        xyz="0 0 0"
-        rpy="0 0 0" />
-      <geometry>
-        <mesh
-          filename="package://stretch_description/meshes/link_gripper_fingertip_right.STL" />
+          filename="package://stretch_description/meshes/link_gripper_fingertip.STL" />
+      </geometry>
+      <material
+        name="">
+        <color
+          rgba="0.25 0.25 0.25 1" />
+      </material>
+    </visual>
+    <collision>
+      <origin
+        xyz="0 0 0"
+        rpy="0 0 0" />
+      <geometry>
+        <mesh
+          filename="package://stretch_description/meshes/collision/link_gripper_fingertip.STL" />
       </geometry>
     </collision>
@@ -263,5 +271,5 @@
     <origin
       xyz="${scale_finger_length * -0.19011} -0.014912 0"
-      rpy="-1.5708 -2.0539E-15 0.58705" />
+      rpy="-${pi/2} 0 0.58705" />
     <parent
       link="link_gripper_finger_right" />

File: stretch_description/urdf/stretch_laser_range_finder.xacro (robot description, xacro)
@@ -36,6 +36,5 @@
         rpy="0 0 0" />
       <geometry>
-        <mesh
-          filename="package://stretch_description/meshes/laser.STL" />
+        <cylinder radius="0.0350" length="0.0195" />
       </geometry>
     </collision>

File: stretch_description/urdf/stretch_main.xacro (robot description, xacro)
@@ -1,5 +1,4 @@
 <?xml version="1.0"?>
 <robot xmlns:xacro="http://www.ros.org/wiki/xacro" name="stretch_main">
-  <xacro:property name="M_PI" value="3.1415926535897931" />
   <xacro:property name="joint_damping" value="21.75"/>
   <xacro:property name="arm_damping" value="21.75"/>
@@ -33,16 +32,16 @@
       </geometry>
       <material
-        name="">
-        <color
-          rgba="0.792156862745098 0.819607843137255 0.933333333333333 1" />
-      </material>
-    </visual>
-    <collision>
-      <origin
-        xyz="0 0 0"
-        rpy="0 0 0" />
-      <geometry>
-        <mesh
-          filename="package://stretch_description/meshes/base_link.STL" />
+        name="LightGray">
+        <color
+          rgba=".74 .74 .78 1" />
+      </material>
+    </visual>
+    <collision>
+      <origin
+        xyz="0 0 0"
+        rpy="0 0 0" />
+      <geometry>
+        <mesh
+          filename="package://stretch_description/meshes/collision/base_link.STL" />
       </geometry>
     </collision>
@@ -52,5 +51,5 @@
     <inertial>
       <origin
-        xyz="1.25554620866719E-07 3.54748938447003E-07 0.0239581106165018"
+        xyz="0 0 0.0239581106165018"
         rpy="0 0 0" />
       <mass
@@ -75,15 +74,13 @@
         name="">
         <color
-          rgba="0.792156862745098 0.819607843137255 0.933333333333333 1" />
-      </material>
-    </visual>
-    <collision>
-      <origin
-        xyz="0 0 0"
-        rpy="0 0 0" />
-      <geometry>
-        <mesh
-          filename="package://stretch_description/meshes/link_right_wheel.STL" />
-          <!-- <cylinder radius="0.051" length="0.0225" /> -->
+          rgba=".13 .13 .13 1" />
+      </material>
+    </visual>
+    <collision>
+      <origin
+        xyz="0 0 0"
+        rpy="0 0 0" />
+      <geometry>
+          <cylinder radius="0.051" length="0.0225" />
       </geometry>
     </collision>
@@ -94,5 +91,5 @@
     <origin
       xyz="-0.00300000000000034 -0.15765 0.0508000000000004"
-      rpy="-1.57079632679489 -1.11022302462516E-16 7.28583859910277E-17" />
+      rpy="-${pi/2} 0 0 " />
     <parent
       link="base_link" />
@@ -107,5 +104,5 @@
     <inertial>
       <origin
-        xyz="1.2555462092223E-07 -3.54748938502514E-07 -0.0239581106165035"
+        xyz="0 0 -0.0239581106165035"
         rpy="0 0 0" />
       <mass
@@ -130,15 +127,13 @@
         name="">
         <color
-          rgba="0.792156862745098 0.819607843137255 0.933333333333333 1" />
-      </material>
-    </visual>
-    <collision>
-      <origin
-        xyz="0 0 0"
-        rpy="0 0 0" />
-      <geometry>
-        <mesh
-          filename="package://stretch_description/meshes/link_left_wheel.STL" />
-        <!-- <cylinder radius="0.051" length="0.0225" /> -->
+          rgba=".13 .13 .13 1" />
+      </material>
+    </visual>
+    <collision>
+      <origin
+        xyz="0 0 0"
+        rpy="0 0 0" />
+      <geometry>
+          <cylinder radius="0.051" length="0.0225" />
       </geometry>
     </collision>
@@ -149,5 +144,5 @@
     <origin
       xyz="-0.00300000000001899 0.15765 0.0507999999999994"
-      rpy="-1.5707963267949 3.16227047920818E-31 7.88745438253713E-16" />
+      rpy="-1.5707963267949 0 0" />
     <parent
       link="base_link" />
@@ -186,5 +181,5 @@
         name="">
         <color
-          rgba="0.792156862745098 0.819607843137255 0.933333333333333 1" />
+          rgba=".13 .13 .13 1" />
       </material>
     </visual>
@@ -204,5 +199,5 @@
     <parent link="base_link"/>
     <child link="caster_link"/>
-    <origin xyz="-0.245 0.0 0.032" rpy="${-M_PI/2} 0 0"/>
+    <origin xyz="-0.245 0.0 0.032" rpy="${-pi/2} 0 0"/>
     <axis xyz="0 0 1" />
   </joint>
@@ -234,14 +229,13 @@
         name="">
         <color
-          rgba="0.792156862745098 0.819607843137255 0.933333333333333 1" />
-      </material>
-    </visual>
-    <collision>
-      <origin
-        xyz="0 0 0"
-        rpy="0 0 0" />
-      <geometry>
-        <mesh
-          filename="package://stretch_description/meshes/link_mast.STL" />
+          rgba=".13 .13 .13 1" />
+      </material>
+    </visual>
+    <collision>
+      <origin
+        xyz="0 0.7075 0"
+        rpy="0 0 0" />
+      <geometry>
+        <box size="0.0384 1.2850 0.0384" />
       </geometry>
     </collision>
@@ -287,14 +281,14 @@
         name="">
         <color
-          rgba="0.792156862745098 0.819607843137255 0.933333333333333 1" />
-      </material>
-    </visual>
-    <collision>
-      <origin
-        xyz="0 0 0"
-        rpy="0 0 0" />
-      <geometry>
-        <mesh
-          filename="package://stretch_description/meshes/link_lift.STL" />
+          rgba=".5 .5 .5 1" />
+      </material>
+    </visual>
+    <collision>
+      <origin
+        xyz="0 0 0"
+        rpy="0 0 0" />
+      <geometry>
+        <mesh
+          filename="package://stretch_description/meshes/collision/link_lift.STL" />
       </geometry>
     </collision>
@@ -305,5 +299,5 @@
     <origin
       xyz="-0.0369217062323472 0.165471199999996 -0.000341653286793524"
-      rpy="-1.57079632679552 1.5615431375292 -6.2942004366467E-13" />
+      rpy="-${pi/2} ${pi/2} 0" />
     <parent
       link="link_mast" />
@@ -322,5 +316,5 @@
     <inertial>
       <origin
-        xyz="-1.61247276464493E-06 1.54715589201215E-06 -0.0953252706040035"
+        xyz="0 0 -0.0953252706040035"
         rpy="0 0 0" />
       <mass
@@ -345,14 +339,13 @@
         name="">
         <color
-          rgba="0.792156862745098 0.819607843137255 0.933333333333333 1" />
-      </material>
-    </visual>
-    <collision>
-      <origin
-        xyz="0 0 0"
-        rpy="0 0 0" />
-      <geometry>
-        <mesh
-          filename="package://stretch_description/meshes/link_arm_l4.STL" />
+          rgba=".13 .13 .13 1" />
+      </material>
+    </visual>
+    <collision>
+      <origin
+        xyz="0 0 -0.1112"
+        rpy="0 0 0" />
+      <geometry>
+        <box size="0.0593 0.0592 0.2225" />
       </geometry>
     </collision>
@@ -363,5 +356,5 @@
     <origin
       xyz="-0.25471 0 0"
-      rpy="1.5708 -3.1019E-16 -1.5708" />
+      rpy="${pi/2} 0 -${pi/2}" />
     <parent
       link="link_lift" />
@@ -376,5 +369,5 @@
     <inertial>
       <origin
-        xyz="-3.34873468621488E-07 4.7411336306924E-07 -0.0974069598289041"
+        xyz="0 0 -0.0974069598289041"
         rpy="0 0 0" />
       <mass
@@ -399,14 +392,13 @@
         name="">
         <color
-          rgba="0.792156862745098 0.819607843137255 0.933333333333333 1" />
-      </material>
-    </visual>
-    <collision>
-      <origin
-        xyz="0 0 0"
-        rpy="0 0 0" />
-      <geometry>
-        <mesh
-          filename="package://stretch_description/meshes/link_arm_l3.STL" />
+          rgba=".13 .13 .13 1" />
+      </material>
+    </visual>
+    <collision>
+      <origin
+        xyz="0 0 -0.1133"
+        rpy="0 0 0" />
+      <geometry>
+        <box size="0.0552 0.0552 0.2265" />
       </geometry>
     </collision>
@@ -417,5 +409,5 @@
     <origin
       xyz="0 0 0.013"
-      rpy="3.5742E-16 3.2123E-16 -2.4565E-16" />
+      rpy="0 0 0" />
     <parent
       link="link_arm_l4" />
@@ -432,5 +424,5 @@
     <inertial>
       <origin
-        xyz="-3.31043560508615E-07 3.13422303999111E-07 -0.097255883541891"
+        xyz="0 0 -0.097255883541891"
         rpy="0 0 0" />
       <mass
@@ -455,14 +447,13 @@
         name="">
         <color
-          rgba="0.792156862745098 0.819607843137255 0.933333333333333 1" />
-      </material>
-    </visual>
-    <collision>
-      <origin
-        xyz="0 0 0"
-        rpy="0 0 0" />
-      <geometry>
-        <mesh
-          filename="package://stretch_description/meshes/link_arm_l2.STL" />
+          rgba=".13 .13 .13 1" />
+      </material>
+    </visual>
+    <collision>
+      <origin
+        xyz="0 0 -0.1133"
+        rpy="0 0 0" />
+      <geometry>
+        <box size="0.0512 0.0512 0.2265" />
       </geometry>
     </collision>
@@ -473,5 +464,5 @@
     <origin
       xyz="0 0 0.013"
-      rpy="2.91385731014123E-16 4.44300759504684E-17 3.25691080516352E-16" />
+      rpy="0 0 0" />
     <parent
       link="link_arm_l3" />
@@ -488,5 +479,5 @@
     <inertial>
       <origin
-        xyz="-3.36876635420591E-07 3.05876091066803E-07 -0.0969117032232756"
+        xyz="0 0 -0.0969117032232756"
         rpy="0 0 0" />
       <mass
@@ -511,14 +502,13 @@
         name="">
         <color
-          rgba="0.792156862745098 0.819607843137255 0.933333333333333 1" />
-      </material>
-    </visual>
-    <collision>
-      <origin
-        xyz="0 0 0"
-        rpy="0 0 0" />
-      <geometry>
-        <mesh
-          filename="package://stretch_description/meshes/link_arm_l1.STL" />
+          rgba=".13 .13 .13 1" />
+      </material>
+    </visual>
+    <collision>
+      <origin
+        xyz="0 0 -0.1133"
+        rpy="0 0 0" />
+      <geometry>
+        <box size="0.0473 0.0472 0.2265"/>
       </geometry>
     </collision>
@@ -529,5 +519,5 @@
     <origin
       xyz="0 0 0.013"
-      rpy="7.41596560408007E-17 1.33876788296791E-16 -2.44545873596083E-16" />
+      rpy="0 0 0" />
     <parent
       link="link_arm_l2" />
@@ -567,14 +557,22 @@
         name="">
         <color
-          rgba="0.792156862745098 0.819607843137255 0.933333333333333 1" />
-      </material>
-    </visual>
-    <collision>
-      <origin
-        xyz="0 0 0"
-        rpy="0 0 0" />
-      <geometry>
-        <mesh
-          filename="package://stretch_description/meshes/link_arm_l0.STL" />
+          rgba=".13 .13 .13 1" />
+      </material>
+    </visual>
+    <collision>
+      <origin
+        xyz="0 0 0"
+        rpy="0 0 0" />
+      <geometry>
+        <mesh
+          filename="package://stretch_description/meshes/collision/link_arm_l0.STL" />
+      </geometry>
+    </collision>
+    <collision>
+      <origin
+        xyz="0.0002 -0.0003 -0.0865"
+        rpy="0 0 0" />
+      <geometry>
+        <box size="0.0457 0.0452 0.2265" />
       </geometry>
     </collision>
@@ -585,5 +583,5 @@
     <origin
       xyz="0 0 -0.0137499999999938"
-      rpy="-3.05317390622457E-16 -4.23236224076729E-16 -2.68425135229209E-17" />
+      rpy="0 0 0" />
     <parent
       link="link_arm_l1" />
@@ -600,5 +598,5 @@
     <inertial>
       <origin
-        xyz="-8.02795716750571E-06 1.93811447768422E-05 0.018946700595851"
+        xyz="0 0 0.018946700595851"
         rpy="0 0 0" />
       <mass
@@ -623,14 +621,13 @@
         name="">
         <color
-	        rgba="0.792156862745098 0.819607843137255 0.933333333333333 1" />
-      </material>
-    </visual>
-    <collision>
-      <origin
-        xyz="0 0 0"
-        rpy="0 0 0" />
-      <geometry>
-        <mesh
-          filename="package://stretch_description/meshes/link_wrist_yaw.STL" />
+	        rgba=".13 .13 .13 1" />
+      </material>
+    </visual>
+    <collision>
+      <origin
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
File: stretch_description/urdf/stretch_respeaker.xacro (robot description, xacro)
@@ -19,5 +19,5 @@
       <origin
         xyz="0 0 0"
-        rpy="0 0 0" />
+        rpy="0 0 ${pi/2}" />
       <geometry>
         <mesh
@@ -27,14 +27,21 @@
         name="">
         <color
-          rgba="0.792156862745098 0.819607843137255 0.933333333333333 1" />
+          rgba=".13 .13 .16 1" />
       </material>
     </visual>
     <collision>
       <origin
-        xyz="0 0 0"
+        xyz="-0.0033 0.0232 -0.0196"
         rpy="0 0 0" />
       <geometry>
-        <mesh
-          filename="package://stretch_description/meshes/link_respeaker.STL" />
+        <box size="0.0635 0.0471 0.0367" />
+      </geometry>
+    </collision>
+    <collision>
+      <origin
+        xyz="0.0001 0.0059 -0.0163"
+        rpy="0 0 0" />
+      <geometry>
+        <cylinder radius="0.0070" length="0.0096" />
       </geometry>
     </collision>
@@ -45,6 +52,6 @@
     <!-- rpy="   ?   rotate_sound_source_direction    ?   " -->
     <origin
-      xyz="1.09074743137871E-05 1.36992 0.00303572796911382"
-      rpy="1.57079632679553 0.0 3.14159265358916" />
+      xyz="0 1.36992 0.00303572796911382"
+      rpy="${pi/2} 0.0 ${pi}" />
     <parent
       link="link_mast" />

Commit message: Increase joint damping
Makes the model behave better with high gain simulation
Reduce needless precision in some masses
Make gripper slightly heavier

File: stretch_description/urdf/stretch_gripper.xacro (robot description, xacro)
@@ -9,5 +9,5 @@
         rpy="0 0 0" />
       <mass
-        value="0.101902711393094" />
+        value="0.45" />
       <inertia
         ixx="0.001"
@@ -126,5 +126,5 @@
         rpy="0 0 0" />
       <mass
-        value="0.00382159917455729" />
+        value="0.01" />
       <inertia
         ixx="0.001"
@@ -179,5 +179,5 @@
         rpy="0 0 0" />
       <mass
-        value="0.0476207785199481" />
+        value="0.05" />
       <inertia
         ixx="0.001"
@@ -233,5 +233,5 @@
         rpy="0 0 0" />
       <mass
-        value="0.00382160037319545" />
+        value="0.01" />
       <inertia
         ixx="0.001"

File: stretch_description/urdf/stretch_main.xacro (robot description, xacro)
@@ -1,8 +1,8 @@
 <?xml version="1.0"?>
 <robot xmlns:xacro="http://www.ros.org/wiki/xacro" name="stretch_main">
-  <xacro:property name="joint_damping" value="21.75"/>
-  <xacro:property name="arm_damping" value="21.75"/>
-  <xacro:property name="joint_friction" value="10.48"/>
-  <xacro:property name="arm_friction" value="2.48"/>
+  <xacro:property name="joint_damping" value="200"/>
+  <xacro:property name="arm_damping" value="200"/>
+  <xacro:property name="joint_friction" value="10"/>
+  <xacro:property name="arm_friction" value="20"/>
   <xacro:property name="joint_spring_stiffness" value="0"/>
   <xacro:property name="joint_spring_reference" value="0"/>
@@ -14,5 +14,5 @@
         rpy="0 0 0" />
       <mass
-        value="12.0" />
+        value="16.0" />
       <inertia
         ixx="0.00013"
@@ -209,5 +209,5 @@
         rpy="0 0 0" />
       <mass
-        value="0.749143203376401" />
+        value="3" />
       <inertia
         ixx="0.000251"
@@ -261,5 +261,5 @@
         rpy="0 0 0" />
       <mass
-        value="0.444820831236007" />
+        value="0.5" />
       <inertia
         ixx="0.000567192946271367"
@@ -309,6 +309,6 @@
   <!--<limit effort="100" lower="0.0" upper="1.095" velocity="1.0"/>-->
   <!-- copied value did not reach the top of mesh model with GUI sliders and RViz -->
-  <limit effort="100" lower="0.0" upper="1.1" velocity="0.5"/>
-  <dynamics friction="40.0" damping="5.0"/>
+  <limit effort="100" lower="0.0" upper="1.1" velocity="0.3"/>
+  <dynamics friction="40.0" damping="200.0"/>
   </joint>
   <link
@@ -319,5 +319,5 @@
         rpy="0 0 0" />
       <mass
-        value="0.0676525455789735" />
+        value="0.07" />
       <inertia
         ixx="0.000122002023066796"
@@ -372,5 +372,5 @@
         rpy="0 0 0" />
       <mass
-        value="0.0626921047058405" />
+        value="0.07" />
       <inertia
         ixx="0.001"
@@ -427,5 +427,5 @@
         rpy="0 0 0" />
       <mass
-        value="0.0569074368576238" />
+        value="0.06" />
       <inertia
         ixx="0.001"
@@ -482,5 +482,5 @@
         rpy="0 0 0" />
       <mass
-        value="0.0511763619538321" />
+        value="0.05" />
       <inertia
         ixx="0.001"
@@ -537,5 +537,5 @@
         rpy="0 0 0" />
       <mass
-        value="0.101241250325294" />
+        value="0.10" />
       <inertia
         ixx="0.001"
@@ -601,5 +601,5 @@
         rpy="0 0 0" />
       <mass
-        value="0.0405398981326229" />
+        value="0.08" />
       <inertia
         ixx="0.001"
@@ -660,5 +660,5 @@
         rpy="0 0 0" />
       <mass
-        value="0.129454717596498" />
+        value="0.13" />
       <inertia
         ixx="0.001"
@@ -713,5 +713,5 @@
         rpy="0 0 0" />
       <mass
-        value="0.035858341182617" />
+        value="0.04" />
       <inertia
         ixx="0.001"
@@ -768,5 +768,5 @@
         rpy="0 0 0" />
       <mass
-        value="0.0701242408063442" />
+        value="0.07" />
       <inertia
         ixx="0.001"
