Commit message: Resolve aruco marker z-fighting
The aruco meshes are just slightly-rounded rects of different sizes, but their normals seem to be messed up causing flickering
Remove these meshes and use manually specified black boxes in the URDF

File: stretch_description/urdf/stretch_aruco.xacro (robot description, xacro)
@@ -5,39 +5,29 @@
     <inertial>
       <origin
-        xyz="0 0 -5.00000000014378E-07"
-        rpy="0 0 0" />
-      <mass
-        value="3.59999999990368E-06" />
-      <inertia
-        ixx="0"
-        ixy="0"
-        ixz="0"
-        iyy="0"
-        iyz="0"
-        izz="0" />
-    </inertial>
-    <visual>
-      <origin
-        xyz="0 0 0"
-        rpy="0 0 0" />
-      <geometry>
-        <mesh
-          filename="package://stretch_description/meshes/link_aruco_right_base.STL" />
-      </geometry>
-      <material
-        name="">
-        <color
-          rgba="0.792156862745098 0.819607843137255 0.933333333333333 1" />
-      </material>
-    </visual>
-    <collision>
-      <origin
-        xyz="0 0 0"
-        rpy="0 0 0" />
-      <geometry>
-        <mesh
-          filename="package://stretch_description/meshes/link_aruco_right_base.STL" />
-      </geometry>
-    </collision>
+        xyz="0 0 0"
+        rpy="0 0 0" />
+      <mass
+        value="0.01" />
+      <inertia
+        ixx="0"
+        ixy="0"
+        ixz="0"
+        iyy="0"
+        iyz="0"
+        izz="0" />
+    </inertial>
+    <visual>
+      <origin
+        xyz="0 0 0"
+        rpy="0 0 0" />
+      <geometry>
+        <box size="0.06 0.06 0.0005"/>
+      </geometry>
+      <material
+        name="">
+        <color
+          rgba="0.0 0.0 0.0 1" />
+      </material>
+    </visual>
   </link>
   <joint
@@ -58,39 +48,29 @@
     <inertial>
       <origin
-        xyz="0 0 -5.00000000014378E-07"
-        rpy="0 0 0" />
-      <mass
-        value="3.59999999990368E-06" />
-      <inertia
-        ixx="0"
-        ixy="0"
-        ixz="0"
-        iyy="0"
-        iyz="0"
-        izz="0" />
-    </inertial>
-    <visual>
-      <origin
-        xyz="0 0 0"
-        rpy="0 0 0" />
-      <geometry>
-        <mesh
-          filename="package://stretch_description/meshes/link_aruco_left_base.STL" />
-      </geometry>
-      <material
-        name="">
-        <color
-          rgba="0.792156862745098 0.819607843137255 0.933333333333333 1" />
-      </material>
-    </visual>
-    <collision>
-      <origin
-        xyz="0 0 0"
-        rpy="0 0 0" />
-      <geometry>
-        <mesh
-          filename="package://stretch_description/meshes/link_aruco_left_base.STL" />
-      </geometry>
-    </collision>
+        xyz="0 0 0"
+        rpy="0 0 0" />
+      <mass
+        value="0.01" />
+      <inertia
+        ixx="0"
+        ixy="0"
+        ixz="0"
+        iyy="0"
+        iyz="0"
+        izz="0" />
+    </inertial>
+    <visual>
+      <origin
+        xyz="0 0 0"
+        rpy="0 0 0" />
+      <geometry>
+        <box size="0.06 0.06 0.0005"/>
+      </geometry>
+      <material
+        name="">
+        <color
+          rgba="0.0 0.0 0.0 1" />
+      </material>
+    </visual>
   </link>
   <joint
@@ -111,5 +91,5 @@
     <inertial>
       <origin
-        xyz="-2.77555756156289E-17 2.56739074444567E-16 -0.000125000000000042"
+        xyz="0 0 0"
         rpy="0 0 0" />
       <mass
@@ -128,22 +108,12 @@
         rpy="0 0 0" />
       <geometry>
-        <mesh
-          filename="package://stretch_description/meshes/link_aruco_shoulder.STL" />
-      </geometry>
-      <material
-        name="">
-        <color
-          rgba="0.792156862745098 0.819607843137255 0.933333333333333 1" />
-      </material>
-    </visual>
-    <collision>
-      <origin
-        xyz="0 0 0"
-        rpy="0 0 0" />
-      <geometry>
-        <mesh
-          filename="package://stretch_description/meshes/link_aruco_shoulder.STL" />
-      </geometry>
-    </collision>
+        <box size="0.04 0.04 0.0005"/>
+      </geometry>
+      <material
+        name="">
+        <color
+          rgba="0.0 0.0 0.0 1" />
+      </material>
+    </visual>
   </link>
   <joint
@@ -152,5 +122,5 @@
     <origin
       xyz="-0.0133768876375287 0.0558540528812078 0.0861368272417975"
-      rpy="-1.53998860117704E-29 3.55962409571165E-15 0.0" />
+      rpy="0.0 0.0 0.0" />
     <parent
       link="link_lift" />
@@ -164,5 +134,5 @@
     <inertial>
       <origin
-        xyz="1.11022302462516E-16 3.05311331771918E-16 -0.00012499999999821"
+        xyz="0 0 0"
         rpy="0 0 0" />
       <mass
@@ -181,22 +151,12 @@
         rpy="0 0 0" />
       <geometry>
-        <mesh
-          filename="package://stretch_description/meshes/link_aruco_top_wrist.STL" />
-      </geometry>
-      <material
-        name="">
-        <color
-          rgba="0.792156862745098 0.819607843137255 0.933333333333333 1" />
-      </material>
-    </visual>
-    <collision>
-      <origin
-        xyz="0 0 0"
-        rpy="0 0 0" />
-      <geometry>
-        <mesh
-          filename="package://stretch_description/meshes/link_aruco_top_wrist.STL" />
-      </geometry>
-    </collision>
+        <box size="0.03 0.03 0.0005"/>
+      </geometry>
+      <material
+        name="">
+        <color
+          rgba="0.0 0.0 0.0 1" />
+      </material>
+    </visual>
   </link>
   <joint
@@ -217,5 +177,5 @@
     <inertial>
       <origin
-        xyz="8.32667268468867E-17 1.77635683940025E-15 -0.000125000000000264"
+        xyz="0 0 0"
         rpy="0 0 0" />
       <mass
@@ -234,22 +194,12 @@
         rpy="0 0 0" />
       <geometry>
-        <mesh
-          filename="package://stretch_description/meshes/link_aruco_inner_wrist.STL" />
-      </geometry>
-      <material
-        name="">
-        <color
-          rgba="0.792156862745098 0.819607843137255 0.933333333333333 1" />
-      </material>
-    </visual>
-    <collision>
-      <origin
-        xyz="0 0 0"
-        rpy="0 0 0" />
-      <geometry>
-        <mesh
-          filename="package://stretch_description/meshes/link_aruco_inner_wrist.STL" />
-      </geometry>
-    </collision>
+        <box size="0.06 0.06 0.0005"/>
+      </geometry>
+      <material
+        name="">
+        <color
+          rgba="0 0 0 1" />
+      </material>
+    </visual>
   </link>
   <joint

Commit message: Fix an oversized aruco marker in URDF

File: stretch_description/urdf/stretch_aruco.xacro (robot description, xacro)
@@ -194,5 +194,5 @@
         rpy="0 0 0" />
       <geometry>
-        <box size="0.06 0.06 0.0005"/>
+        <box size="0.03 0.03 0.0005"/>
       </geometry>
       <material

Commit message: integrating hello robot noetic changes and moveit_config

File: stretch_description/urdf/stretch_aruco.xacro (robot description, xacro)
@@ -5,29 +5,39 @@
     <inertial>
       <origin
-        xyz="0 0 0"
-        rpy="0 0 0" />
-      <mass
-        value="0.01" />
-      <inertia
-        ixx="0"
-        ixy="0"
-        ixz="0"
-        iyy="0"
-        iyz="0"
-        izz="0" />
-    </inertial>
-    <visual>
-      <origin
-        xyz="0 0 0"
-        rpy="0 0 0" />
-      <geometry>
-        <box size="0.06 0.06 0.0005"/>
-      </geometry>
-      <material
-        name="">
-        <color
-          rgba="0.0 0.0 0.0 1" />
-      </material>
-    </visual>
+        xyz="0 0 -5.00000000014378E-07"
+        rpy="0 0 0" />
+      <mass
+        value="3.59999999990368E-06" />
+      <inertia
+        ixx="0"
+        ixy="0"
+        ixz="0"
+        iyy="0"
+        iyz="0"
+        izz="0" />
+    </inertial>
+    <visual>
+      <origin
+        xyz="0 0 0"
+        rpy="0 0 0" />
+      <geometry>
+        <mesh
+          filename="package://stretch_description/meshes/link_aruco_right_base.STL" />
+      </geometry>
+      <material
+        name="">
+        <color
+          rgba="0.792156862745098 0.819607843137255 0.933333333333333 1" />
+      </material>
+    </visual>
+    <collision>
+      <origin
+        xyz="0 0 0"
+        rpy="0 0 0" />
+      <geometry>
+        <mesh
+          filename="package://stretch_description/meshes/link_aruco_right_base.STL" />
+      </geometry>
+    </collision>
   </link>
   <joint
@@ -48,29 +58,39 @@
     <inertial>
       <origin
-        xyz="0 0 0"
-        rpy="0 0 0" />
-      <mass
-        value="0.01" />
-      <inertia
-        ixx="0"
-        ixy="0"
-        ixz="0"
-        iyy="0"
-        iyz="0"
-        izz="0" />
-    </inertial>
-    <visual>
-      <origin
-        xyz="0 0 0"
-        rpy="0 0 0" />
-      <geometry>
-        <box size="0.06 0.06 0.0005"/>
-      </geometry>
-      <material
-        name="">
-        <color
-          rgba="0.0 0.0 0.0 1" />
-      </material>
-    </visual>
+        xyz="0 0 -5.00000000014378E-07"
+        rpy="0 0 0" />
+      <mass
+        value="3.59999999990368E-06" />
+      <inertia
+        ixx="0"
+        ixy="0"
+        ixz="0"
+        iyy="0"
+        iyz="0"
+        izz="0" />
+    </inertial>
+    <visual>
+      <origin
+        xyz="0 0 0"
+        rpy="0 0 0" />
+      <geometry>
+        <mesh
+          filename="package://stretch_description/meshes/link_aruco_left_base.STL" />
+      </geometry>
+      <material
+        name="">
+        <color
+          rgba="0.792156862745098 0.819607843137255 0.933333333333333 1" />
+      </material>
+    </visual>
+    <collision>
+      <origin
+        xyz="0 0 0"
+        rpy="0 0 0" />
+      <geometry>
+        <mesh
+          filename="package://stretch_description/meshes/link_aruco_left_base.STL" />
+      </geometry>
+    </collision>
   </link>
   <joint
@@ -91,5 +111,5 @@
     <inertial>
       <origin
-        xyz="0 0 0"
+        xyz="-2.77555756156289E-17 2.56739074444567E-16 -0.000125000000000042"
         rpy="0 0 0" />
       <mass
@@ -108,12 +128,22 @@
         rpy="0 0 0" />
       <geometry>
-        <box size="0.04 0.04 0.0005"/>
-      </geometry>
-      <material
-        name="">
-        <color
-          rgba="0.0 0.0 0.0 1" />
-      </material>
-    </visual>
+        <mesh
+          filename="package://stretch_description/meshes/link_aruco_shoulder.STL" />
+      </geometry>
+      <material
+        name="">
+        <color
+          rgba="0.792156862745098 0.819607843137255 0.933333333333333 1" />
+      </material>
+    </visual>
+    <collision>
+      <origin
+        xyz="0 0 0"
+        rpy="0 0 0" />
+      <geometry>
+        <mesh
+          filename="package://stretch_description/meshes/link_aruco_shoulder.STL" />
+      </geometry>
+    </collision>
   </link>
   <joint
@@ -122,5 +152,5 @@
     <origin
       xyz="-0.0133768876375287 0.0558540528812078 0.0861368272417975"
-      rpy="0.0 0.0 0.0" />
+      rpy="-1.53998860117704E-29 3.55962409571165E-15 0.0" />
     <parent
       link="link_lift" />
@@ -134,5 +164,5 @@
     <inertial>
       <origin
-        xyz="0 0 0"
+        xyz="1.11022302462516E-16 3.05311331771918E-16 -0.00012499999999821"
         rpy="0 0 0" />
       <mass
@@ -151,12 +181,22 @@
         rpy="0 0 0" />
       <geometry>
-        <box size="0.03 0.03 0.0005"/>
-      </geometry>
-      <material
-        name="">
-        <color
-          rgba="0.0 0.0 0.0 1" />
-      </material>
-    </visual>
+        <mesh
+          filename="package://stretch_description/meshes/link_aruco_top_wrist.STL" />
+      </geometry>
+      <material
+        name="">
+        <color
+          rgba="0.792156862745098 0.819607843137255 0.933333333333333 1" />
+      </material>
+    </visual>
+    <collision>
+      <origin
+        xyz="0 0 0"
+        rpy="0 0 0" />
+      <geometry>
+        <mesh
+          filename="package://stretch_description/meshes/link_aruco_top_wrist.STL" />
+      </geometry>
+    </collision>
   </link>
   <joint
@@ -177,5 +217,5 @@
     <inertial>
       <origin
-        xyz="0 0 0"
+        xyz="8.32667268468867E-17 1.77635683940025E-15 -0.000125000000000264"
         rpy="0 0 0" />
       <mass
@@ -194,12 +234,22 @@
         rpy="0 0 0" />
       <geometry>
-        <box size="0.03 0.03 0.0005"/>
-      </geometry>
-      <material
-        name="">
-        <color
-          rgba="0 0 0 1" />
-      </material>
-    </visual>
+        <mesh
+          filename="package://stretch_description/meshes/link_aruco_inner_wrist.STL" />
+      </geometry>
+      <material
+        name="">
+        <color
+          rgba="0.792156862745098 0.819607843137255 0.933333333333333 1" />
+      </material>
+    </visual>
+    <collision>
+      <origin
+        xyz="0 0 0"
+        rpy="0 0 0" />
+      <geometry>
+        <mesh
+          filename="package://stretch_description/meshes/link_aruco_inner_wrist.STL" />
+      </geometry>
+    </collision>
   </link>
   <joint

File: stretch_description/urdf/stretch_gripper.xacro (robot description, xacro)
@@ -9,5 +9,5 @@
         rpy="0 0 0" />
       <mass
-        value="0.45" />
+        value="0.101902711393094" />
       <inertia
         ixx="0.001"
@@ -29,22 +29,14 @@
         name="">
         <color
-          rgba=".13 .13 .16 1" />
-      </material>
-    </visual>
-    <collision>
-      <origin
-        xyz="0 0 0"
-        rpy="0 0 0" />
-      <geometry>
-        <mesh
-          filename="package://stretch_description/meshes/collision/link_gripper.STL" />
-      </geometry>
-    </collision>
-    <collision>
-      <origin
-        xyz="-0.0039 0.0139 -0.0289"
-        rpy="0 0 0" />
-      <geometry>
-        <box size="0.0423 0.0618 0.0578" />
+          rgba="0.792156862745098 0.819607843137255 0.933333333333333 1" />
+      </material>
+    </visual>
+    <collision>
+      <origin
+        xyz="0 0 0"
+        rpy="0 0 0" />
+      <geometry>
+        <mesh
+          filename="package://stretch_description/meshes/link_gripper.STL" />
       </geometry>
     </collision>
@@ -57,5 +49,5 @@
     <origin
       xyz="0 0 0"
-      rpy="3.14159 0 -${pi/2}" />
+      rpy="3.14159 0 -1.5708" />
     <parent
       link="link_wrist_yaw" />
@@ -69,5 +61,5 @@
     <inertial>
       <origin
-        xyz="0.0945047483510102 0.0124301080924361 0"
+        xyz="0.0945047483510102 0.0124301080924361 -4.44089209850063E-16"
         rpy="0 0 0" />
       <mass
@@ -92,5 +84,5 @@
         name="">
         <color
-          rgba="0.8 .8 .8 1" />
+          rgba="0.792156862745098 0.819607843137255 0.933333333333333 1" />
       </material>
     </visual>
@@ -110,5 +102,5 @@
     <origin
       xyz="-0.047231 -0.010151 -0.04679"
-      rpy="0 0.5236 3.1416" />
+      rpy="2.1762E-15 0.5236 3.1416" />
     <parent
       link="link_gripper" />
@@ -123,37 +115,37 @@
     <inertial>
       <origin
-        xyz="0 0 0.00812579670381812"
-        rpy="0 0 0" />
-      <mass
-        value="0.01" />
-      <inertia
-        ixx="0.001"
-        ixy="0"
-        ixz="0"
-        iyy="0.001"
-        iyz="0"
-        izz="0.001" />
-    </inertial>
-    <visual>
-      <origin
-        xyz="0 0 0"
-        rpy="0 0 0" />
-      <geometry>
-        <mesh
-          filename="package://stretch_description/meshes/link_gripper_fingertip.STL" />
-      </geometry>
-      <material
-        name="">
-        <color
-          rgba="0.25 0.25 0.25 1" />
-      </material>
-    </visual>
-    <collision>
-      <origin
-        xyz="0 0 0"
-        rpy="0 0 0" />
-      <geometry>
-        <mesh
-          filename="package://stretch_description/meshes/collision/link_gripper_fingertip.STL" />
+        xyz="-3.16381381648689E-08 -2.91408530639359E-09 0.00812579670381812"
+        rpy="0 0 0" />
+      <mass
+        value="0.00382159917455729" />
+      <inertia
+        ixx="0.001"
+        ixy="0"
+        ixz="0"
+        iyy="0.001"
+        iyz="0"
+        izz="0.001" />
+    </inertial>
+    <visual>
+      <origin
+        xyz="0 0 0"
+        rpy="0 0 0" />
+      <geometry>
+        <mesh
+          filename="package://stretch_description/meshes/link_gripper_fingertip_left.STL" />
+      </geometry>
+      <material
+        name="">
+        <color
+          rgba="0.250980392156863 0.250980392156863 0.250980392156863 1" />
+      </material>
+    </visual>
+    <collision>
+      <origin
+        xyz="0 0 0"
+        rpy="0 0 0" />
+      <geometry>
+        <mesh
+          filename="package://stretch_description/meshes/link_gripper_fingertip_left.STL" />
       </geometry>
     </collision>
@@ -164,5 +156,5 @@
     <origin
       xyz="${scale_finger_length * 0.19011} 0.014912 0"
-      rpy="-${pi/2} 0 -2.5545" />
+      rpy="-1.5708 -4.774E-15 -2.5545" />
     <parent
       link="link_gripper_finger_left" />
@@ -179,5 +171,5 @@
         rpy="0 0 0" />
       <mass
-        value="0.05" />
+        value="0.0476207785199481" />
       <inertia
         ixx="0.001"
@@ -199,5 +191,5 @@
         name="">
         <color
-          rgba=".8 .8 .8 1" />
+          rgba="0.792156862745098 0.819607843137255 0.933333333333333 1" />
       </material>
     </visual>
@@ -217,5 +209,5 @@
     <origin
       xyz="-0.047231 0.010049 -0.04679"
-      rpy="3.1416 -0.5236 0" />
+      rpy="3.1416 -0.5236 1.2943E-15" />
     <parent
       link="link_gripper" />
@@ -230,37 +222,37 @@
     <inertial>
       <origin
-        xyz="0 0 0.00812579516130402"
-        rpy="0 0 0" />
-      <mass
-        value="0.01" />
-      <inertia
-        ixx="0.001"
-        ixy="0"
-        ixz="0"
-        iyy="0.001"
-        iyz="0"
-        izz="0.001" />
-    </inertial>
-    <visual>
-      <origin
-        xyz="0 0 0"
-        rpy="0 0 0" />
-      <geometry>
-        <mesh
-          filename="package://stretch_description/meshes/link_gripper_fingertip.STL" />
-      </geometry>
-      <material
-        name="">
-        <color
-          rgba="0.25 0.25 0.25 1" />
-      </material>
-    </visual>
-    <collision>
-      <origin
-        xyz="0 0 0"
-        rpy="0 0 0" />
-      <geometry>
-        <mesh
-          filename="package://stretch_description/meshes/collision/link_gripper_fingertip.STL" />
+        xyz="2.59386303963494E-08 6.70949018566347E-09 0.00812579516130402"
+        rpy="0 0 0" />
+      <mass
+        value="0.00382160037319545" />
+      <inertia
+        ixx="0.001"
+        ixy="0"
+        ixz="0"
+        iyy="0.001"
+        iyz="0"
+        izz="0.001" />
+    </inertial>
+    <visual>
+      <origin
+        xyz="0 0 0"
+        rpy="0 0 0" />
+      <geometry>
+        <mesh
+          filename="package://stretch_description/meshes/link_gripper_fingertip_right.STL" />
+      </geometry>
+      <material
+        name="">
+        <color
+          rgba="0.250980392156863 0.250980392156863 0.250980392156863 1" />
+      </material>
+    </visual>
+    <collision>
+      <origin
+        xyz="0 0 0"
+        rpy="0 0 0" />
+      <geometry>
+        <mesh
+          filename="package://stretch_description/meshes/link_gripper_fingertip_right.STL" />
       </geometry>
     </collision>
@@ -271,5 +263,5 @@
     <origin
       xyz="${scale_finger_length * -0.19011} -0.014912 0"
-      rpy="-${pi/2} 0 0.58705" />
+      rpy="-1.5708 -2.0539E-15 0.58705" />
     <parent
       link="link_gripper_finger_right" />

File: stretch_description/urdf/stretch_laser_range_finder.xacro (robot description, xacro)
@@ -36,5 +36,6 @@
         rpy="0 0 0" />
       <geometry>
-        <cylinder radius="0.0350" length="0.0195" />
+        <mesh
+          filename="package://stretch_description/meshes/laser.STL" />
       </geometry>
     </collision>
