Commit message: integrating hello robot noetic changes and moveit_config

File: stretch_description/urdf/stretch_main.xacro (robot description, xacro)
@@ -1,8 +1,7 @@
 <?xml version="1.0"?>
 <robot xmlns:xacro="http://www.ros.org/wiki/xacro" name="stretch_main">
-  <xacro:property name="joint_damping" value="200"/>
-  <xacro:property name="arm_damping" value="200"/>
-  <xacro:property name="joint_friction" value="10"/>
-  <xacro:property name="arm_friction" value="20"/>
+  <xacro:property name="M_PI" value="3.1415926535897931" />
+  <xacro:property name="joint_damping" value="21.75"/>
+  <xacro:property name="joint_friction" value="10.48"/>
   <xacro:property name="joint_spring_stiffness" value="0"/>
   <xacro:property name="joint_spring_reference" value="0"/>
@@ -14,12 +13,12 @@
         rpy="0 0 0" />
       <mass
-        value="16.0" />
-      <inertia
-        ixx="0.00013"
-        ixy="0"
-        ixz="0"
-        iyy="0.00012"
-        iyz="0"
-        izz="0.000218" />
+        value="1.0723782659782" />
+      <inertia
+        ixx="0.00310580907710135"
+        ixy="1.5182848191076E-06"
+        ixz="0.00041690466732394"
+        iyy="0.00433798719991832"
+        iyz="1.33487716258445E-05"
+        izz="0.0037204727467362" />
     </inertial>
     <visual>
@@ -32,16 +31,16 @@
       </geometry>
       <material
-        name="LightGray">
-        <color
-          rgba=".74 .74 .78 1" />
-      </material>
-    </visual>
-    <collision>
-      <origin
-        xyz="0 0 0"
-        rpy="0 0 0" />
-      <geometry>
-        <mesh
-          filename="package://stretch_description/meshes/collision/base_link.STL" />
+        name="">
+        <color
+          rgba="0.792156862745098 0.819607843137255 0.933333333333333 1" />
+      </material>
+    </visual>
+    <collision>
+      <origin
+        xyz="0 0 0"
+        rpy="0 0 0" />
+      <geometry>
+        <mesh
+          filename="package://stretch_description/meshes/base_link.STL" />
       </geometry>
     </collision>
@@ -51,5 +50,5 @@
     <inertial>
       <origin
-        xyz="0 0 0.0239581106165018"
+        xyz="1.25554620866719E-07 3.54748938447003E-07 0.0239581106165018"
         rpy="0 0 0" />
       <mass
@@ -74,13 +73,14 @@
         name="">
         <color
-          rgba=".13 .13 .13 1" />
-      </material>
-    </visual>
-    <collision>
-      <origin
-        xyz="0 0 0"
-        rpy="0 0 0" />
-      <geometry>
-          <cylinder radius="0.051" length="0.0225" />
+          rgba="0.792156862745098 0.819607843137255 0.933333333333333 1" />
+      </material>
+    </visual>
+    <collision>
+      <origin
+        xyz="0 0 0"
+        rpy="0 0 0" />
+      <geometry>
+        <mesh
+          filename="package://stretch_description/meshes/link_right_wheel.STL" />
       </geometry>
     </collision>
@@ -91,5 +91,5 @@
     <origin
       xyz="-0.00300000000000034 -0.15765 0.0508000000000004"
-      rpy="-${pi/2} 0 0 " />
+      rpy="-1.57079632679489 -1.11022302462516E-16 7.28583859910277E-17" />
     <parent
       link="base_link" />
@@ -104,5 +104,5 @@
     <inertial>
       <origin
-        xyz="0 0 -0.0239581106165035"
+        xyz="1.2555462092223E-07 -3.54748938502514E-07 -0.0239581106165035"
         rpy="0 0 0" />
       <mass
@@ -127,13 +127,14 @@
         name="">
         <color
-          rgba=".13 .13 .13 1" />
-      </material>
-    </visual>
-    <collision>
-      <origin
-        xyz="0 0 0"
-        rpy="0 0 0" />
-      <geometry>
-          <cylinder radius="0.051" length="0.0225" />
+          rgba="0.792156862745098 0.819607843137255 0.933333333333333 1" />
+      </material>
+    </visual>
+    <collision>
+      <origin
+        xyz="0 0 0"
+        rpy="0 0 0" />
+      <geometry>
+        <mesh
+          filename="package://stretch_description/meshes/link_left_wheel.STL" />
       </geometry>
     </collision>
@@ -144,5 +145,5 @@
     <origin
       xyz="-0.00300000000001899 0.15765 0.0507999999999994"
-      rpy="-1.5707963267949 0 0" />
+      rpy="-1.5707963267949 3.16227047920818E-31 7.88745438253713E-16" />
     <parent
       link="base_link" />
@@ -181,5 +182,5 @@
         name="">
         <color
-          rgba=".13 .13 .13 1" />
+          rgba="0.792156862745098 0.819607843137255 0.933333333333333 1" />
       </material>
     </visual>
@@ -199,5 +200,5 @@
     <parent link="base_link"/>
     <child link="caster_link"/>
-    <origin xyz="-0.245 0.0 0.032" rpy="${-pi/2} 0 0"/>
+    <origin xyz="-0.245 0.0 0.032" rpy="${-M_PI/2} 0 0"/>
     <axis xyz="0 0 1" />
   </joint>
@@ -206,15 +207,15 @@
     <inertial>
       <origin
-        xyz="0 0.7073971284176834 0"
-        rpy="0 0 0" />
-      <mass
-        value="3" />
-      <inertia
-        ixx="0.000251"
-        ixy="0"
-        ixz="-0"
-        iyy="0.000000"
-        iyz="0"
-        izz="0.000251" />
+        xyz="0.00755818572975822 0.773971284176834 0.00647313086620024"
+        rpy="0 0 0" />
+      <mass
+        value="0.749143203376401" />
+      <inertia
+        ixx="0.0709854511954588"
+        ixy="-0.00433428742758457"
+        ixz="-0.000186110788697573"
+        iyy="0.000437922053342648"
+        iyz="-0.00288788257713431"
+        izz="0.071104808501661" />
     </inertial>
     <visual>
@@ -229,13 +230,14 @@
         name="">
         <color
-          rgba=".13 .13 .13 1" />
-      </material>
-    </visual>
-    <collision>
-      <origin
-        xyz="0 0.7075 0"
-        rpy="0 0 0" />
-      <geometry>
-        <box size="0.0384 1.2850 0.0384" />
+          rgba="0.792156862745098 0.819607843137255 0.933333333333333 1" />
+      </material>
+    </visual>
+    <collision>
+      <origin
+        xyz="0 0 0"
+        rpy="0 0 0" />
+      <geometry>
+        <mesh
+          filename="package://stretch_description/meshes/link_mast.STL" />
       </geometry>
     </collision>
@@ -261,5 +263,5 @@
         rpy="0 0 0" />
       <mass
-        value="0.5" />
+        value="0.444820831236007" />
       <inertia
         ixx="0.000567192946271367"
@@ -281,14 +283,14 @@
         name="">
         <color
-          rgba=".5 .5 .5 1" />
-      </material>
-    </visual>
-    <collision>
-      <origin
-        xyz="0 0 0"
-        rpy="0 0 0" />
-      <geometry>
-        <mesh
-          filename="package://stretch_description/meshes/collision/link_lift.STL" />
+          rgba="0.792156862745098 0.819607843137255 0.933333333333333 1" />
+      </material>
+    </visual>
+    <collision>
+      <origin
+        xyz="0 0 0"
+        rpy="0 0 0" />
+      <geometry>
+        <mesh
+          filename="package://stretch_description/meshes/link_lift.STL" />
       </geometry>
     </collision>
@@ -299,5 +301,5 @@
     <origin
       xyz="-0.0369217062323472 0.165471199999996 -0.000341653286793524"
-      rpy="-${pi/2} ${pi/2} 0" />
+      rpy="-1.57079632679552 1.5615431375292 -6.2942004366467E-13" />
     <parent
       link="link_mast" />
@@ -309,6 +311,5 @@
   <!--<limit effort="100" lower="0.0" upper="1.095" velocity="1.0"/>-->
   <!-- copied value did not reach the top of mesh model with GUI sliders and RViz -->
-  <limit effort="100" lower="0.0" upper="1.1" velocity="0.3"/>
-  <dynamics friction="40.0" damping="200.0"/>
+  <limit effort="100" lower="0.0" upper="1.1" velocity="1.0"/>
   </joint>
   <link
@@ -316,8 +317,8 @@
     <inertial>
       <origin
-        xyz="0 0 -0.0953252706040035"
-        rpy="0 0 0" />
-      <mass
-        value="0.07" />
+        xyz="-1.61247276464493E-06 1.54715589201215E-06 -0.0953252706040035"
+        rpy="0 0 0" />
+      <mass
+        value="0.0676525455789735" />
       <inertia
         ixx="0.000122002023066796"
@@ -339,13 +340,14 @@
         name="">
         <color
-          rgba=".13 .13 .13 1" />
-      </material>
-    </visual>
-    <collision>
-      <origin
-        xyz="0 0 -0.1112"
-        rpy="0 0 0" />
-      <geometry>
-        <box size="0.0593 0.0592 0.2225" />
+          rgba="0.792156862745098 0.819607843137255 0.933333333333333 1" />
+      </material>
+    </visual>
+    <collision>
+      <origin
+        xyz="0 0 0"
+        rpy="0 0 0" />
+      <geometry>
+        <mesh
+          filename="package://stretch_description/meshes/link_arm_l4.STL" />
       </geometry>
     </collision>
@@ -356,5 +358,5 @@
     <origin
       xyz="-0.25471 0 0"
-      rpy="${pi/2} 0 -${pi/2}" />
+      rpy="1.5708 -3.1019E-16 -1.5708" />
     <parent
       link="link_lift" />
@@ -363,5 +365,4 @@
     <axis
       xyz="0 0 0" />
-    <dynamics damping="${arm_damping}" friction="${arm_friction}" />
   </joint>
   <link
@@ -369,8 +370,8 @@
     <inertial>
       <origin
-        xyz="0 0 -0.0974069598289041"
-        rpy="0 0 0" />
-      <mass
-        value="0.07" />
+        xyz="-3.34873468621488E-07 4.7411336306924E-07 -0.0974069598289041"
+        rpy="0 0 0" />
+      <mass
+        value="0.0626921047058405" />
       <inertia
         ixx="0.001"
@@ -392,13 +393,14 @@
         name="">
         <color
-          rgba=".13 .13 .13 1" />
-      </material>
-    </visual>
-    <collision>
-      <origin
-        xyz="0 0 -0.1133"
-        rpy="0 0 0" />
-      <geometry>
-        <box size="0.0552 0.0552 0.2265" />
+          rgba="0.792156862745098 0.819607843137255 0.933333333333333 1" />
+      </material>
+    </visual>
+    <collision>
+      <origin
+        xyz="0 0 0"
+        rpy="0 0 0" />
+      <geometry>
+        <mesh
+          filename="package://stretch_description/meshes/link_arm_l3.STL" />
       </geometry>
     </collision>
@@ -409,5 +411,5 @@
     <origin
       xyz="0 0 0.013"
-      rpy="0 0 0" />
+      rpy="3.5742E-16 3.2123E-16 -2.4565E-16" />
     <parent
       link="link_arm_l4" />
@@ -417,6 +419,5 @@
 	xyz="0 0 1" />
     <!-- 0.13 = 0.52/4-->
-    <limit effort="100" lower="0.0" upper="0.13" velocity="0.1"/>
-    <dynamics damping="${arm_damping}" friction="${arm_friction}" />
+    <limit effort="100" lower="0.0" upper="0.13" velocity="1.0"/>
   </joint>
   <link
@@ -424,8 +425,8 @@
     <inertial>
       <origin
-        xyz="0 0 -0.097255883541891"
-        rpy="0 0 0" />
-      <mass
-        value="0.06" />
+        xyz="-3.31043560508615E-07 3.13422303999111E-07 -0.097255883541891"
+        rpy="0 0 0" />
+      <mass
+        value="0.0569074368576238" />
       <inertia
         ixx="0.001"
@@ -447,13 +448,14 @@
         name="">
         <color
-          rgba=".13 .13 .13 1" />
-      </material>
-    </visual>
-    <collision>
-      <origin
-        xyz="0 0 -0.1133"
-        rpy="0 0 0" />
-      <geometry>
-        <box size="0.0512 0.0512 0.2265" />
+          rgba="0.792156862745098 0.819607843137255 0.933333333333333 1" />
+      </material>
+    </visual>
+    <collision>
+      <origin
+        xyz="0 0 0"
+        rpy="0 0 0" />
+      <geometry>
+        <mesh
+          filename="package://stretch_description/meshes/link_arm_l2.STL" />
       </geometry>
     </collision>
@@ -464,5 +466,5 @@
     <origin
       xyz="0 0 0.013"
-      rpy="0 0 0" />
+      rpy="2.91385731014123E-16 4.44300759504684E-17 3.25691080516352E-16" />
     <parent
       link="link_arm_l3" />
@@ -472,6 +474,5 @@
 	xyz="0 0 1" />
     <!-- 0.13 = 0.52/4-->
-    <limit effort="100" lower="0.0" upper="0.13" velocity="0.1"/>
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
File: stretch_description/urdf/stretch_respeaker.xacro (robot description, xacro)
@@ -19,5 +19,5 @@
       <origin
         xyz="0 0 0"
-        rpy="0 0 ${pi/2}" />
+        rpy="0 0 0" />
       <geometry>
         <mesh
@@ -27,21 +27,14 @@
         name="">
         <color
-          rgba=".13 .13 .16 1" />
+          rgba="0.792156862745098 0.819607843137255 0.933333333333333 1" />
       </material>
     </visual>
     <collision>
       <origin
-        xyz="-0.0033 0.0232 -0.0196"
+        xyz="0 0 0"
         rpy="0 0 0" />
       <geometry>
-        <box size="0.0635 0.0471 0.0367" />
-      </geometry>
-    </collision>
-    <collision>
-      <origin
-        xyz="0.0001 0.0059 -0.0163"
-        rpy="0 0 0" />
-      <geometry>
-        <cylinder radius="0.0070" length="0.0096" />
+        <mesh
+          filename="package://stretch_description/meshes/link_respeaker.STL" />
       </geometry>
     </collision>
@@ -52,6 +45,6 @@
     <!-- rpy="   ?   rotate_sound_source_direction    ?   " -->
     <origin
-      xyz="0 1.36992 0.00303572796911382"
-      rpy="${pi/2} 0.0 ${pi}" />
+      xyz="1.09074743137871E-05 1.36992 0.00303572796911382"
+      rpy="1.57079632679553 0.0 3.14159265358916" />
     <parent
       link="link_mast" />

File: stretch_gazebo/urdf/stretch_gazebo.urdf.xacro (robot description, xacro)
@@ -1,4 +1,4 @@
 <?xml version="1.0"?>
-<robot xmlns:xacro="http://www.ros.org/wiki/xacro" name="stretch_description">
+<robot xmlns:xacro="http://www.ros.org/wiki/xacro" name="stretch">
   <xacro:arg name="gpu_lidar" default="false" />
   <xacro:arg name="visualize_lidar" default="false" />
@@ -10,9 +10,6 @@
   <xacro:include filename="$(find stretch_description)/urdf/stretch_gripper.xacro" />
   <gazebo>
-    <plugin name="gazebo_ros_control" filename="libstretch_gazebo_ros_control_plugin.so">
-      <robotSimType>stretch_gazebo/StretchHardwareGazebo</robotSimType>
+    <plugin name="gazebo_ros_control" filename="libgazebo_ros_control.so">
       <robotNamespace>/</robotNamespace>
-      <eStopTopic>estop</eStopTopic>
-      <jointStatesTopic>stretch/joint_states</jointStatesTopic>
     </plugin>
   </gazebo>
@@ -352,5 +349,5 @@
     </actuator>
     <joint name="joint_lift">
-      <hardwareInterface>hardware_interface/EffortJointInterface</hardwareInterface>
+      <hardwareInterface>hardware_interface/PositionJointInterface</hardwareInterface>
     </joint>
   </transmission>
@@ -402,5 +399,5 @@
     </actuator>
     <joint name="joint_arm_l0">
-      <hardwareInterface>hardware_interface/EffortJointInterface</hardwareInterface>
+      <hardwareInterface>hardware_interface/PositionJointInterface</hardwareInterface>
     </joint>
   </transmission>
@@ -411,5 +408,5 @@
     </actuator>
     <joint name="joint_arm_l1">
-      <hardwareInterface>hardware_interface/EffortJointInterface</hardwareInterface>
+      <hardwareInterface>hardware_interface/PositionJointInterface</hardwareInterface>
     </joint>
   </transmission>
@@ -420,5 +417,5 @@
     </actuator>
     <joint name="joint_arm_l2">
-      <hardwareInterface>hardware_interface/EffortJointInterface</hardwareInterface>
+      <hardwareInterface>hardware_interface/PositionJointInterface</hardwareInterface>
     </joint>
   </transmission>
@@ -429,5 +426,5 @@
     </actuator>
     <joint name="joint_arm_l3">
-      <hardwareInterface>hardware_interface/EffortJointInterface</hardwareInterface>
+      <hardwareInterface>hardware_interface/PositionJointInterface</hardwareInterface>
     </joint>
   </transmission>
@@ -447,5 +444,5 @@
     </actuator>
     <joint name="joint_wrist_yaw">
-      <hardwareInterface>hardware_interface/EffortJointInterface</hardwareInterface>
+      <hardwareInterface>hardware_interface/PositionJointInterface</hardwareInterface>
     </joint>
   </transmission>
@@ -478,5 +475,5 @@
     </actuator>
     <joint name="joint_head_pan">
-      <hardwareInterface>hardware_interface/EffortJointInterface</hardwareInterface>
+      <hardwareInterface>hardware_interface/PositionJointInterface</hardwareInterface>
     </joint>
   </transmission>
@@ -487,5 +484,5 @@
     </actuator>
     <joint name="joint_head_tilt">
-      <hardwareInterface>hardware_interface/EffortJointInterface</hardwareInterface>
+      <hardwareInterface>hardware_interface/PositionJointInterface</hardwareInterface>
     </joint>
   </transmission>
@@ -545,5 +542,5 @@
     </actuator>
     <joint name="joint_gripper_finger_left">
-      <hardwareInterface>hardware_interface/EffortJointInterface</hardwareInterface>
+      <hardwareInterface>hardware_interface/PositionJointInterface</hardwareInterface>
     </joint>
   </transmission>
@@ -554,19 +551,6 @@
     </actuator>
     <joint name="joint_gripper_finger_right">
-      <hardwareInterface>hardware_interface/EffortJointInterface</hardwareInterface>
-    </joint>
-  </transmission>
-  <!-- Ground Truth Odom plugin -->
-  <gazebo>
-    <plugin name="p3d_base_controller" filename="libgazebo_ros_p3d.so">
-      <alwaysOn>true</alwaysOn>
-      <updateRate>25.0</updateRate>
-      <bodyName>base_link</bodyName>
-      <topicName>ground_truth</topicName>
-      <gaussianNoise>0.01</gaussianNoise>
-      <frameName>world</frameName>
-      <xyzOffsets>0 0 0</xyzOffsets>
-      <rpyOffsets>0 0 0</rpyOffsets>
-    </plugin>
-  </gazebo>
+      <hardwareInterface>hardware_interface/PositionJointInterface</hardwareInterface>
+    </joint>
+</transmission>
 </robot>
